Commit message: Gazebo

File: src/mycobot_ros2/mycobot_description/urdf/control/gazebo_sim_ros2_control.urdf.xacro (robot description, xacro)
@@ -1,10 +1,23 @@
 <?xml version="1.0" ?>
+<!-- 机器人模型根标签，声明xacro命名空间 -->
 <robot xmlns:xacro="http://wiki.ros.org/xacro">
+    <!-- 定义宏：加载Gazebo仿真ros2_control插件 -->
+    <!-- 参数：
+         robot_name: 机器人名称，用于定位控制器yaml配置文件
+         use_gazebo: 布尔开关，true才加载Gazebo插件，RViz离线可视化时不加载
+    -->
     <xacro:macro name="load_gazebo_sim_ros2_control_plugin" params="robot_name use_gazebo">
+        <!-- 条件判断：仅当use_gazebo为true时，才生成Gazebo插件代码 -->
         <xacro:if value="${use_gazebo}">
+            <!-- Gazebo专属标签，内部配置Gazebo仿真插件 -->
             <gazebo>
+                <!-- gz_ros2_control插件：在Gazebo中对接ros2_control控制器框架 -->
+                <!-- filename：插件库文件名；name：插件类名 -->
                 <plugin filename="gz_ros2_control-system" name="gz_ros2_control::GazeboSimROS2ControlPlugin">
+                    <!-- 控制器参数文件路径，ros2_control从中读取关节控制器配置 -->
                     <parameters>$(find mycobot_moveit2_config)/config/${robot_name}/ros2_controllers.yaml</parameters>
+                    <!-- ROS2话题重映射 -->
                     <ros>
+                        <!-- 重映射：controller_manager读取的robot_description，使用全局/robot_description -->
                         <remapping>/controller_manager/robot_description:=/robot_description</remapping>
                     </ros>

File: src/mycobot_ros2/mycobot_description/urdf/mech/g_shape_base_v2_0.urdf.xacro (robot description, xacro)
@@ -1,9 +1,79 @@
 <?xml version="1.0" ?>
+<!--
+    声明这是一个 Xacro 文件。
+    Xacro 是 ROS 中用于生成 URDF 的 XML 宏语言，
+    可以通过 macro、参数、变量等方式复用机器人模型代码。
+-->
 <robot xmlns:xacro="http://wiki.ros.org/xacro">
+    <!--
+        定义一个名为 g_shape_base 的 Xacro 宏。
+        参数：
+        1. base_link：基础 Link 的名称，例如 base_link
+        2. prefix：Link 名称前缀，例如 robot1_、robot2_
+        调用这个宏后，会生成：
+            <link name="${prefix}${base_link}">
+        例如：
+            prefix = robot1_
+            base_link = base_link
+        最终 Link 名称就是：
+            robot1_base_link
+    -->
     <xacro:macro name="g_shape_base" params="base_link prefix">
+        <!--
+            定义机器人底座的 Link。
+            ${prefix}${base_link}
+            表示把 prefix 和 base_link 拼接起来。
+            例如：
+                prefix = ""
+                base_link = base_link
+                -> base_link
+            或：
+                prefix = robot1_
+                base_link = base_link
+                -> robot1_base_link
+        -->
         <link name="${prefix}${base_link}">
+            <!--
+                inertial：定义这个 Link 的动力学 / 惯性属性。
+                Gazebo 进行物理仿真时，需要知道物体的：
+                - 质量
+                - 质心位置
+                - 惯性矩阵
+                如果机器人需要在 Gazebo 中进行真实物理运动，
+                inertial 信息非常重要。
+            -->
             <inertial>
+                <!--
+                    定义惯性坐标系相对于 Link 坐标系的位置和姿态。
+                    xyz="0 0 0.0"
+                    表示惯性参考点位于 Link 原点。
+                    rpy="0 0 0"
+                    表示惯性坐标系没有旋转。
+                -->
                 <origin xyz="0 0 0.0" rpy="0 0 0"/>
+                <!--
+                    定义这个 Link 的质量。
+                    单位：
+                        kg
+                    这里表示底座质量为：
+                        0.33 kg
+                -->
                 <mass value="0.33"/>
+                <!--
+                    定义惯性张量。
+                    惯性张量描述物体对于绕不同坐标轴旋转的惯性。
+                    矩阵形式为：
+                        | ixx  ixy  ixz |
+                        | ixy  iyy  iyz |
+                        | ixz  iyz  izz |
+                    其中：
+                        ixx：绕 X 轴的转动惯量
+                        iyy：绕 Y 轴的转动惯量
+                        izz：绕 Z 轴的转动惯量
+                        ixy、ixz、iyz：
+                        表示不同坐标轴之间的惯性耦合项。
+                    单位通常为：
+                        kg·m²
+                -->
                 <inertia
                     ixx="0.000784" ixy="0.0" ixz="0.0"
@@ -11,22 +81,141 @@
                     izz="0.001598"/>
             </inertial>
+            <!--
+                visual：定义机器人在 RViz / Gazebo 中
+                "看起来是什么样子"。
+                visual 主要负责显示模型，
+                不直接决定物理碰撞。
+            -->
             <visual>
+                <!--
+                    geometry：定义可视化几何形状。
+                -->
                 <geometry>
-                    <mesh filename="file://$(find mycobot_description)/meshes/g_shape_base_v2_0/visual/base_link.dae"/>
+                    <!--
+                        mesh：使用外部网格模型作为底座的视觉模型。
+                        filename：
+                        指定 mesh 文件的位置。
+                        file://
+                        表示使用文件系统中的本地文件。
+                        $(find mycobot_description)
+                        表示查找 ROS 2/ROS 中
+                        mycobot_description 功能包的位置。
+                        最终找到：
+                            meshes/g_shape_base_v2_0/visual/base_link.dae
+                        .dae：
+                        COLLADA 格式的 3D 模型文件。
+                        注意：
+                        这里的 mesh 主要用于显示，
+                        下面 collision 才负责碰撞检测。
+                    -->
+                    <mesh
+                        filename="file://$(find mycobot_description)/meshes/g_shape_base_v2_0/visual/base_link.dae"/>
                 </geometry>
+                <!--
+                    设置 visual 模型相对于 Link 坐标系的位置和姿态。
+                    xyz="0.0 0 -0.03"
+                    表示：
+                        X：0
+                        Y：0
+                        Z：-0.03 m
+                    即视觉模型沿 Z 轴向下移动 3 cm。
+                    rpy="0 0 ${pi/2}"
+                    表示：
+                        Roll  = 0
+                        Pitch = 0
+                        Yaw   = π/2
+                    即绕 Z 轴旋转 90°。
+                    ${pi/2}
+                    是 Xacro 表达式，表示 π/2。
+                -->
                 <origin xyz="0.0 0 -0.03" rpy="0 0 ${pi/2}"/>
             </visual>
+            <!--
+                collision：定义这个 Link 用于物理碰撞检测的几何模型。
+                它和 visual 是分开的：
+                    visual
+                    -> 负责"看起来什么样"
+                    collision
+                    -> 负责"物理上碰到什么"
+                这里没有使用复杂的 DAE 网格，
+                而是使用简单的 Box 碰撞模型。
+                这样可以降低 Gazebo 物理计算的复杂度。
+            -->
             <collision>
+                <!--
+                    geometry：定义碰撞模型的几何形状。
+                -->
                 <geometry>
+                    <!--
+                        使用一个长方体作为碰撞模型。
+                        size="0.105 0.14 0.02"
+                        分别表示：
+                            X = 0.105 m
+                            Y = 0.14  m
+                            Z = 0.02  m
+                        即：
+                            10.5 cm × 14 cm × 2 cm
+                    -->
                     <box size="0.105 0.14 0.02"/>
                 </geometry>
+                <!--
+                    设置碰撞模型相对于 Link 坐标系的位置。
+                    xyz="0.0 0.0 -0.015"
+                    表示碰撞盒沿 Z 轴向下移动：
+                        0.015 m = 1.5 cm
+                    rpy="0 0 0"
+                    表示碰撞盒没有旋转。
+                -->
                 <origin xyz="0.0 0.0 -0.015" rpy="0 0 0"/>
             </collision>
         </link>
+        <!--
+            gazebo：Gazebo 专用配置。
+            reference="${prefix}${base_link}"
+            表示：
+            当前 Gazebo 配置作用于哪个 Link。
+            这里引用的就是前面创建的：
+                ${prefix}${base_link}
+            例如：
+                robot1_base_link
+        -->
         <gazebo reference="${prefix}${base_link}">
+            <!--
+                visual：
+                对 Gazebo 中这个 Link 的视觉显示进行额外配置。
+                注意：
+                这里不是重新定义 visual 几何模型，
+                而是在 Gazebo 中对已经存在的 visual
+                添加 Gazebo 专用属性。
+            -->
             <visual>
+                <!--
+                    material：设置 Gazebo 中模型的材质属性。
+                -->
                 <material>
+                    <!--
+                        。
+                        RGBA：
+                            R = 0.5
+                            G = 0.5
+                            B = 0.5
+                            A = 1
+                        即灰色，不透明。
+                    -->
                     <ambient>0.5 0.5 0.5 1</ambient>
+                    <!--
+                        diffuse：
+                        漫反射颜色。
+                        这里同样设置为灰色。
+                    -->
                     <diffuse>0.5 0.5 0.5 1</diffuse>
+                    <!--
+                        specular：
+                        镜面反射颜色。
+                        数值越明显，
+                        模型受到光照时的高光效果通常越明显。
+                        这里设置为：
+                            0.5 0.5 0.5 1
+                    -->
                     <specular>0.5 0.5 0.5 1</specular>
                 </material>

File: src/mycobot_ros2/mycobot_description/urdf/mech/mycobot_280_arm.urdf.xacro (robot description, xacro)
@@ -1,19 +1,36 @@
 <?xml version="1.0"?>
 <robot xmlns:xacro="http://www.ros.org/wiki/xacro">
+  <!-- xacro 内部变量 -->
+  <!-- 1. 关节最大力矩(N·m)，用于 joint limit 限制 -->
   <xacro:property name="joint_effort" value="56.0"/>
+  <!-- 2. 关节最大角速度(rad/s)，用于 joint limit 限制 -->
   <xacro:property name="joint_velocity" value="2.792527"/>
+  <!-- 3. 关节阻尼系数，Gazebo 动力学 dynamics 标签使用 -->
   <xacro:property name="joint_damping" value="0.0"/>
+  <!-- 4. 关节库伦摩擦系数，Gazebo 动力学 dynamics 标签使用 -->
   <xacro:property name="joint_friction" value="0.0"/>
+  <!-- 1. 连杆 1 质量，单位 kg，用于 inertial 惯性参数 -->
   <xacro:property name="link1_mass" value="0.12"/>
+  <!-- 2. 连杆 2 质量，单位 kg，用于 inertial 惯性参数 -->
   <xacro:property name="link2_mass" value="0.19"/>
+  <!-- 3. 连杆 3 质量，单位 kg，用于 inertial 惯性参数 -->
   <xacro:property name="link3_mass" value="0.16"/>
+  <!-- 4. 连杆 4 质量，单位 kg，用于 inertial 惯性参数 -->
   <xacro:property name="link4_mass" value="0.124"/>
+  <!-- 5. 连杆 5 质量，单位 kg，用于 inertial 惯性参数 -->
   <xacro:property name="link5_mass" value="0.11"/>
+  <!-- 6. 连杆 6 质量，单位 kg，用于 inertial 惯性参数 -->
   <xacro:property name="link6_mass" value="0.0739"/>
+  <!-- 7. 末端法兰 质量，单位 kg，用于 inertial 惯性参数 -->
   <xacro:property name="flange_mass" value="0.035"/>
+  <!-- 定义宏：生成连杆惯性块，快速复用 inertial 标签 -->
   <xacro:macro name="link_inertial" params="mass ixx iyy izz">
+    <!-- 惯性参数块，Gazebo 物理仿真必需，描述连杆质量与惯量 -->
     <inertial>
+      <!-- 惯性坐标系原点，相对于连杆本体坐标系，rpy 姿态角 -->
       <origin xyz="0 0 0.0" rpy="0 0 0"/>
+      <!-- 连杆质量 -->
       <mass value="${mass}"/>
+      <!-- 惯性张量矩阵，简化模型：非对角惯量 ixy,ixz,iyz 全部置 0 -->
       <inertia
         ixx="${ixx}" ixy="0.0" ixz="0.0"
@@ -22,10 +39,23 @@
     </inertial>
   </xacro:macro>
+  <!-- 定义宏：给Gazebo中指定连杆设置视觉材质（仅Gazebo仿真生效，不影响URDF可视化） -->
+  <!-- 参数：
+     ref_link: 目标连杆名称，gazebo标签的reference，指定要修改材质的link
+     ambient: 环境光颜色，RGBA四元组，取值0~1
+     diffuse: 漫反射颜色，RGBA四元组，物体本身基础颜色
+     specular: 高光反射颜色，RGBA四元组，控制反光亮点颜色
+  -->
   <xacro:macro name="material_visual" params="ref_link ambient diffuse specular">
+    <!-- Gazebo专属标签，reference指定作用的link，只在Gazebo仿真器识别 -->
     <gazebo reference="${ref_link}">
-      <visual>
+      <!-- Gazebo内的视觉渲染配置，和URDF的visual相互独立 -->
+      <visual>
+        <!-- 材质定义块 -->
         <material>
+          <!-- 环境光颜色，环境照射到物体上的基础底色 RGBA -->
           <ambient>${ambient}</ambient>
+          <!-- 漫反射颜色，物体受光呈现的主体颜色 RGBA -->
           <diffuse>${diffuse}</diffuse>
+          <!-- 高光颜色，光源直射产生的反光亮点 RGBA -->
           <specular>${specular}</specular>
         </material>
@@ -33,22 +63,39 @@
     </gazebo>
   </xacro:macro>
+  <!-- 定义宏：Mycobot280机械臂主体模型，批量生成所有连杆+关节，支持多实例前缀、自定义底座与末端法兰 -->
+  <!-- 参数说明：
+       base_link: 底座连杆名称，作为机械臂根部父连杆
+       flange_link: 末端法兰连杆名称
+       prefix: 连杆/关节名称前缀，用于在同一个urdf中加载多台机械臂，避免命名冲突
+       *origin: 可变参数块，用于传入固定关节的origin标签，适配底座安装位姿
+  -->
   <xacro:macro name="mycobot_280_arm" params="base_link flange_link prefix *origin">
+    <!-- 1号连杆 -->
     <link name="${prefix}link1">
+      <!-- 调用惯性宏，填入link1质量与惯量张量对角元 -->
       <xacro:link_inertial mass="${link1_mass}" ixx="0.000148" iyy="0.000148" izz="0.000096"/>
-      <visual>
+      <!-- RViz可视化几何体 -->
+      <visual>
+        <!-- 使用dae网格模型作为外观 -->
         <geometry>
           <mesh filename="file://$(find mycobot_description)/meshes/mycobot_280/visual/link1.dae"/>
         </geometry>
+        <!-- 网格相对于link本体坐标系的偏移与旋转 -->
         <origin xyz="0.0 0 0" rpy="0 0 ${-pi/2}"/>
       </visual>
+      <!-- 碰撞检测几何体(Gazebo/碰撞检测用，简化包围盒，比mesh快很多) -->
       <collision>
         <geometry>
           <box size="0.08 0.12 0.075"/>
         </geometry>
+        <!-- 碰撞包围盒相对于link本体坐标系的位姿 -->
         <origin xyz="0.0 -0.01 0.034" rpy="0 0 0"/>
       </collision>
     </link>
+    <!-- 2号连杆 -->
     <link name="${prefix}link2">
+      <!-- 调用惯性宏，填入link2质量与惯量张量对角元 -->
       <xacro:link_inertial mass="${link2_mass}" ixx="0.000148" iyy="0.000148" izz="0.000096"/>
+      <!-- RViz可视化几何体 -->
       <visual>
         <geometry>
@@ -57,4 +104,5 @@
         <origin xyz="0.0 0 -0.06096" rpy="0 0 ${-pi/2}"/>
       </visual>
+      <!-- 碰撞几何体：圆柱简化包围体 -->
       <collision>
         <geometry>
@@ -64,6 +112,9 @@
       </collision>
     </link>
+    <!-- 3号连杆 -->
     <link name="${prefix}link3">
+      <!-- 调用惯性宏，填入link3质量与惯量张量对角元 -->
       <xacro:link_inertial mass="${link3_mass}" ixx="0.000148" iyy="0.000148" izz="0.000096"/>
+      <!-- RViz可视化几何体 -->
       <visual>
         <geometry>
@@ -72,4 +123,5 @@
         <origin xyz="0.0 0 0.03256" rpy="0 ${-pi/2} 0"/>
       </visual>
+      <!-- 碰撞几何体：圆柱简化包围体 -->
       <collision>
         <geometry>
@@ -79,6 +131,9 @@
       </collision>
     </link>
+    <!-- 4号连杆 -->
     <link name="${prefix}link4">
+      <!-- 调用惯性宏，填入link4质量与惯量张量对角元 -->
       <xacro:link_inertial mass="${link4_mass}" ixx="0.000103" iyy="0.000103" izz="0.000096"/>
+      <!-- RViz可视化几何体 -->
       <visual>
         <geometry>
@@ -87,4 +142,5 @@
         <origin xyz="0.0 0 0.03056" rpy="0 ${-pi/2} 0"/>
       </visual>
+      <!-- 碰撞几何体：圆柱简化包围体 -->
       <collision>
         <geometry>
@@ -94,6 +150,9 @@
       </collision>
     </link>
+    <!-- 5号连杆 -->
     <link name="${prefix}link5">
+      <!-- 调用惯性宏，填入link5质量与惯量张量对角元 -->
       <xacro:link_inertial mass="${link5_mass}" ixx="0.000103" iyy="0.000103" izz="0.000096"/>
+      <!-- RViz可视化几何体 -->
       <visual>
         <geometry>
@@ -102,4 +161,5 @@
         <origin xyz="0.0 0 -0.03356" rpy="${-pi/2} 0 0"/>
       </visual>
+      <!-- 碰撞几何体：长方体包围盒 -->
       <collision>
         <geometry>
@@ -109,6 +169,9 @@
       </collision>
     </link>
+    <!-- 6号连杆 -->
     <link name="${prefix}link6">
+      <!-- 调用惯性宏，填入link6质量与惯量张量对角元 -->
       <xacro:link_inertial mass="${link6_mass}" ixx="0.00006649" iyy="0.00006649" izz="0.000096"/>
+      <!-- RViz可视化几何体 -->
       <visual>
         <geometry>
@@ -117,4 +180,5 @@
         <origin xyz="0 0.00 -0.038" rpy="0 0 0"/>
       </visual>
+      <!-- 碰撞几何体：圆柱简化包围体 -->
       <collision>
         <geometry>
@@ -124,6 +188,9 @@
       </collision>
     </link>
+    <!-- 末端法兰连杆 -->
     <link name="${prefix}${flange_link}">
+      <!-- 调用惯性宏，填入末端法兰质量与惯量张量对角元 -->
       <xacro:link_inertial mass="${flange_mass}" ixx="0.0000149" iyy="0.0000149" izz="0.0000196"/>
+      <!-- RViz可视化几何体 -->
       <visual>
         <geometry>
@@ -132,4 +199,5 @@
         <origin xyz="0.0 0 -0.012" rpy="0 0 0"/>
       </visual>
+      <!-- 碰撞几何体：小圆柱包围体 -->
       <collision>
         <geometry>
@@ -139,17 +207,27 @@
       </collision>
     </link>
+    <!-- 底座到link1固定关节，用于把机械臂挂载到基座上 -->
     <joint name="${prefix}${base_link}_to_${prefix}link1" type="fixed">
+      <!-- 父连杆：底座 -->
       <parent link="${prefix}${base_link}"/>
+      <!-- 子连杆：1号连杆 -->
       <child link="${prefix}link1"/>
+      <!-- 插入外部传入的origin块，自定义底座安装偏移 -->
       <xacro:insert_block name="origin"/>
     </joint>
+    <!-- J1：link1 -> link2 旋转关节，机械臂第1个转动轴 -->
     <joint name="${prefix}link1_to_${prefix}link2" type="revolute">
-      <axis xyz="0 0 1"/>
+      <!-- 旋转轴方向向量，在父连杆坐标系下 -->
+      <axis xyz="0 0 1"/>
+      <!-- 关节限位：最大力矩、角度上下限、最大角速度 -->
       <limit effort="${joint_effort}" lower="-2.879793" upper="2.879793" velocity="${joint_velocity}"/>
       <parent link="${prefix}link1"/>
       <child link="${prefix}link2"/>
+      <!-- 子连杆相对于父连杆的位姿 -->
       <origin xyz="0 0 0.13156" rpy="0 0 ${pi/2}"/>
-      <dynamics damping="${joint_damping}" friction="${joint_friction}"/>
-    </joint>
+      <!-- 动力学参数：阻尼、库伦摩擦，Gazebo仿真使用 -->
+      <dynamics damping="${joint_damping}" friction="${joint_friction}"/>
+    </joint>
+    <!-- J2：link2 -> link3 旋转关节，机械臂第2个转动轴 -->
     <joint name="${prefix}link2_to_${prefix}link3" type="revolute">
       <axis xyz="0 0 1"/>
@@ -160,4 +238,5 @@
       <dynamics damping="${joint_damping}" friction="${joint_friction}"/>
     </joint>
+    <!-- J3：link3 -> link4 旋转关节，机械臂第3个转动轴 -->
     <joint name="${prefix}link3_to_${prefix}link4" type="revolute">
       <axis xyz="0 0 1"/>
@@ -168,4 +247,5 @@
       <dynamics damping="${joint_damping}" friction="${joint_friction}"/>
     </joint>
+    <!-- J4：link4 -> link5 旋转关节，机械臂第4个转动轴 -->
     <joint name="${prefix}link4_to_${prefix}link5" type="revolute">
       <axis xyz="0 0 1"/>
@@ -176,4 +256,5 @@
       <dynamics damping="${joint_damping}" friction="${joint_friction}"/>
     </joint>
+    <!-- J5：link5 -> link6 旋转关节，机械臂第5个转动轴 -->
     <joint name="${prefix}link5_to_${prefix}link6" type="revolute">
       <axis xyz="0 0 1"/>
@@ -184,6 +265,8 @@
       <dynamics damping="${joint_damping}" friction="${joint_friction}"/>
     </joint>
+    <!-- J6：link6 -> 末端法兰 旋转关节，机械臂第6个转动轴 -->
     <joint name="${prefix}link6_to_${prefix}${flange_link}" type="revolute">
       <axis xyz="0 0 1"/>
+      <!-- J6单独角度限位，和前面J1~J5范围不同 -->
       <limit effort="${joint_effort}" lower="-3.05" upper="3.05" velocity="${joint_velocity}"/>
       <parent link="${prefix}link6"/>
@@ -192,10 +275,17 @@
       <dynamics damping="${joint_damping}" friction="${joint_friction}"/>
     </joint>
+    <!-- 调用材质宏：Gazebo渲染，设置link1材质颜色 -->
     <xacro:material_visual ref_link="${prefix}link1" ambient="0.5 0.5 0.5 1" diffuse="0.5 0.5 0.5 1" specular="0.5 0.5 0.5 1"/>
+    <!-- 调用材质宏：Gazebo渲染，设置link2材质颜色 -->
     <xacro:material_visual ref_link="${prefix}link2" ambient="1 1 1 1" diffuse="1 1 1 1" specular="1 1 1 1"/>
+    <!-- 调用材质宏：Gazebo渲染，设置link3材质颜色 -->
     <xacro:material_visual ref_link="${prefix}link3" ambient="1 1 1 1" diffuse="1 1 1 1" specular="1 1 1 1"/>
+    <!-- 调用材质宏：Gazebo渲染，设置link4材质颜色 -->
     <xacro:material_visual ref_link="${prefix}link4" ambient="1 1 1 1" diffuse="1 1 1 1" specular="1 1 1 1"/>
+    <!-- 调用材质宏：Gazebo渲染，设置link5材质颜色 -->
     <xacro:material_visual ref_link="${prefix}link5" ambient="1 1 1 1" diffuse="1 1 1 1" specular="1 1 1 1"/>
+    <!-- 调用材质宏：Gazebo渲染，设置link6材质颜色 -->
     <xacro:material_visual ref_link="${prefix}link6" ambient="1 1 1 1" diffuse="1 1 1 1" specular="1 1 1 1"/>
+    <!-- 调用材质宏：Gazebo渲染，设置末端法兰材质颜色 -->
     <xacro:material_visual ref_link="${prefix}${flange_link}" ambient="0.5 0.5 0.5 1" diffuse="0.5 0.5 0.5 1" specular="0.5 0.5 0.5 1"/>
   </xacro:macro>
