Commit message: Gazebo

File: src/mycobot_ros2/mycobot_description/urdf/mech/adaptive_gripper.urdf.xacro (robot description, xacro)
@@ -1,202 +1,251 @@
 <?xml version="1.0"?>
+<!-- Xacro命名空间声明，启用xacro宏、变量、参数替换功能 -->
 <robot xmlns:xacro="http://www.ros.org/wiki/xacro">
-  <xacro:property name="joint_effort" value="56.0"/>
-  <xacro:property name="joint_velocity" value="2.792527"/>
-  <xacro:property name="joint_damping" value="0.0"/>
-  <xacro:property name="joint_friction" value="0.0"/>
-  <xacro:property name="gripper_link_mass" value="0.007"/>
-  <xacro:property name="gripper_link_ixx" value="1e-6"/>
-  <xacro:property name="gripper_link_iyy" value="1e-6"/>
-  <xacro:property name="gripper_link_izz" value="1e-6"/>
-  <xacro:macro name="gripper_link_inertial">
-    <inertial>
-      <origin xyz="0 0 0.0" rpy="0 0 0"/>
-      <mass value="${gripper_link_mass}"/>
-      <inertia
-        ixx="${gripper_link_ixx}" ixy="0.0" ixz="0.0"
-        iyy="${gripper_link_iyy}" iyz="0.0"
-        izz="${gripper_link_izz}"/>
-    </inertial>
-  </xacro:macro>
-  <xacro:macro name="adaptive_gripper" params="parent prefix *origin">
-    <link name="${prefix}gripper_base">
-      <inertial>
-        <origin xyz="0 0 0.0" rpy="0 0 0"/>
-        <mass value="0.07"/>
-        <inertia
-          ixx="0.000010725" ixy="0.0" ixz="0.0"
-          iyy="0.000014392" iyz="0.0"
-          izz="0.000018517"/>
-      </inertial>
-      <visual>
-        <geometry>
-          <mesh filename="file://$(find mycobot_description)/meshes/adaptive_gripper/visual/gripper_base.dae"/>
-        </geometry>
-        <origin xyz="0.0 0.0 -0.012" rpy="0 0 0"/>
-      </visual>
-      <collision>
-        <geometry>
-          <box size="0.065 0.025 0.025"/>
-        </geometry>
-        <origin xyz="0.0 0.0 0.0" rpy="0 0 0"/>
-      </collision>
-    </link>
-    <joint name="${prefix}${parent}_to_${prefix}gripper_base" type="fixed">
-      <parent link="${prefix}${parent}"/>
-      <child link="${prefix}gripper_base"/>
-      <xacro:insert_block name="origin"/>
-    </joint>
-    <link name="${prefix}gripper_left1">
-      <xacro:gripper_link_inertial/>
-      <visual>
-        <geometry>
-          <mesh filename="file://$(find mycobot_description)/meshes/adaptive_gripper/visual/gripper_left1.dae"/>
-        </geometry>
-        <origin xyz="0.039 -0.0133 -0.012" rpy="0 0 0"/>
-      </visual>
-      <collision>
-        <geometry>
-          <box size="0.013 0.02 0.015"/>
-        </geometry>
-        <origin xyz="0.013 0.042 -0.010" rpy="0 0 0"/>
-      </collision>
-    </link>
-    <link name="${prefix}gripper_left2">
-      <xacro:gripper_link_inertial/>
-      <visual>
-        <geometry>
-          <mesh filename="file://$(find mycobot_description)/meshes/adaptive_gripper/visual/gripper_left2.dae"/>
-        </geometry>
-        <origin xyz="0.005 -0.0195 -0.012" rpy="0 0 0"/>
-      </visual>
-      <collision>
-        <geometry>
-          <box size="0.02 0.02 0.02"/>
-        </geometry>
-        <origin xyz="-0.025 0.0 -0.010" rpy="0 0 0"/>
-      </collision>
-    </link>
-    <link name="${prefix}gripper_left3">
-      <xacro:gripper_link_inertial/>
-      <visual>
-        <geometry>
-          <mesh filename="file://$(find mycobot_description)/meshes/adaptive_gripper/visual/gripper_left3.dae"/>
-        </geometry>
-        <origin xyz="0.012 0.0025 -0.012" rpy="0 0 0"/>
-      </visual>
-      <collision>
-        <geometry>
-          <box size="0.01 0.01 0.01"/>
-        </geometry>
-        <origin xyz="-0.014 0.005 0.005" rpy="0 0 0"/>
-      </collision>
-    </link>
-    <link name="${prefix}gripper_right1">
-      <xacro:gripper_link_inertial/>
-      <visual>
-        <geometry>
-          <mesh filename="file://$(find mycobot_description)/meshes/adaptive_gripper/visual/gripper_right1.dae"/>
-        </geometry>
-        <origin xyz="-0.039 -0.0133 -0.012" rpy="0 0 0"/>
-      </visual>
-      <collision>
-        <geometry>
-          <box size="0.013 0.02 0.015"/>
-        </geometry>
-        <origin xyz="-0.013 0.042 -0.010" rpy="0 0 0"/>
-      </collision>
-    </link>
-    <link name="${prefix}gripper_right2">
-      <xacro:gripper_link_inertial/>
-      <visual>
-        <geometry>
-          <mesh filename="file://$(find mycobot_description)/meshes/adaptive_gripper/visual/gripper_right2.dae"/>
-        </geometry>
-        <origin xyz="-0.005 -0.0195 -0.012" rpy="0 0 0"/>
-      </visual>
-      <collision>
-        <geometry>
-          <box size="0.02 0.02 0.02"/>
-        </geometry>
-        <origin xyz="0.025 0.0 -0.010" rpy="0 0 0"/>
-      </collision>
-    </link>
-    <link name="${prefix}gripper_right3">
-      <xacro:gripper_link_inertial/>
-      <visual>
-        <geometry>
-          <mesh filename="file://$(find mycobot_description)/meshes/adaptive_gripper/visual/gripper_right3.dae"/>
-        </geometry>
-        <origin xyz="-0.012 0.0025 -0.012" rpy="0 0 0"/>
-      </visual>
-      <collision>
-        <geometry>
-          <box size="0.01 0.01 0.01"/>
-        </geometry>
-        <origin xyz="0.014 0.005 0.005" rpy="0 0 0"/>
-      </collision>
-    </link>
-    <joint name="${prefix}gripper_controller" type="revolute">
-      <axis xyz="0 0 1"/>
-      <limit effort="${joint_effort}" lower="-0.7" upper="0.15" velocity="${joint_velocity}"/>
-      <parent link="${prefix}gripper_base"/>
-      <child link="${prefix}gripper_left3"/>
-      <origin xyz="-0.012 0.005 0" rpy="0 0 0"/>
-      <dynamics damping="${joint_damping}" friction="${joint_friction}"/>
-    </joint>
-    <joint name="${prefix}gripper_base_to_${prefix}gripper_left2" type="revolute">
-      <axis xyz="0 0 1"/>
-      <limit effort="${joint_effort}" lower="-0.8" upper="0.5" velocity="${joint_velocity}"/>
-      <parent link="${prefix}gripper_base"/>
-      <child link="${prefix}gripper_left2"/>
-      <origin xyz="-0.005 0.027 0" rpy="0 0 0"/>
-      <mimic joint="${prefix}gripper_controller" multiplier="1.0" offset="0"/>
-      <dynamics damping="${joint_damping}" friction="${joint_friction}"/>
-    </joint>
-    <joint name="${prefix}gripper_left3_to_${prefix}gripper_left1" type="revolute">
-      <axis xyz="0 0 1"/>
-      <limit effort="${joint_effort}" lower="-0.5" upper="0.5" velocity="${joint_velocity}"/>
-      <parent link="${prefix}gripper_left3"/>
-      <child link="${prefix}gripper_left1"/>
-      <origin xyz="-0.027 0.016 0" rpy="0 0 0"/>
-      <mimic joint="${prefix}gripper_controller" multiplier="-1.0" offset="0"/>
-      <dynamics damping="${joint_damping}" friction="${joint_friction}"/>
-    </joint>
-    <joint name="${prefix}gripper_base_to_${prefix}gripper_right3" type="revolute">
-      <axis xyz="0 0 1"/>
-      <limit effort="${joint_effort}" lower="-0.15" upper="0.7" velocity="${joint_velocity}"/>
-      <parent link="${prefix}gripper_base"/>
-      <child link="${prefix}gripper_right3"/>
-      <origin xyz="0.012 0.005 0" rpy="0 0 0"/>
-      <mimic joint="${prefix}gripper_controller" multiplier="-1.0" offset="0"/>
-      <dynamics damping="${joint_damping}" friction="${joint_friction}"/>
-    </joint>
-    <joint name="${prefix}gripper_base_to_${prefix}gripper_right2" type="revolute">
-      <axis xyz="0 0 1"/>
-      <limit effort="${joint_effort}" lower="-0.5" upper="0.8" velocity="${joint_velocity}"/>
-      <parent link="${prefix}gripper_base"/>
-      <child link="${prefix}gripper_right2"/>
-      <origin xyz="0.005 0.027 0" rpy="0 0 0"/>
-      <mimic joint="${prefix}gripper_controller" multiplier="-1.0" offset="0"/>
-      <dynamics damping="${joint_damping}" friction="${joint_friction}"/>
-    </joint>
-    <joint name="${prefix}gripper_right3_to_${prefix}gripper_right1" type="revolute">
-      <axis xyz="0 0 1"/>
-      <limit effort="${joint_effort}" lower="-0.5" upper="0.5" velocity="${joint_velocity}"/>
-      <parent link="${prefix}gripper_right3"/>
-      <child link="${prefix}gripper_right1"/>
-      <origin xyz="0.027 0.016 0" rpy="0 0 0"/>
-      <mimic joint="${prefix}gripper_controller" multiplier="1.0" offset="0"/>
-      <dynamics damping="${joint_damping}" friction="${joint_friction}"/>
-    </joint>
-    <gazebo reference="${prefix}gripper_base">
-      <visual>
-        <material>
-          <ambient>1 1 1 1</ambient>
-          <diffuse>1 1 1 1</diffuse>
-          <specular>1 1 1 1</specular>
-        </material>
-      </visual>
-    </gazebo>
-  </xacro:macro>
+    <!-- ===================== 全局参数定义 ===================== -->
+    <!-- 关节最大力矩(N·m)：关节能输出的最大扭矩，Gazebo/ros2_control用于力矩限幅 -->
+    <xacro:property name="joint_effort" value="56.0"/>
+    <!-- 关节最大角速度(rad/s)，限制关节运动速度上限 -->
+    <xacro:property name="joint_velocity" value="2.792527"/>
+    <!-- 关节阻尼系数，阻尼会抵抗关节运动，0表示无阻尼 -->
+    <xacro:property name="joint_damping" value="0.0"/>
+    <!-- 关节静摩擦系数，0表示无摩擦，仿真时更容易运动 -->
+    <xacro:property name="joint_friction" value="0.0"/>
+    <!-- 夹爪手指连杆惯性参数：单根手指连杆质量(kg) -->
+    <xacro:property name="gripper_link_mass" value="0.007"/>
+    <!-- 转动惯量，Ixx, Iyy, Izz，单位 kg·m²；对角惯性，非对角项ixy/ixz/iyz=0，代表连杆质心坐标系和惯性主轴重合 -->
+    <xacro:property name="gripper_link_ixx" value="1e-6"/>
+    <xacro:property name="gripper_link_iyy" value="1e-6"/>
+    <xacro:property name="gripper_link_izz" value="1e-6"/>
+    <!-- ===================== 宏：手指连杆惯性块模板 ===================== -->
+    <!-- 复用宏：所有手指小段(gripper_left1/left2...)共用同一套惯性配置，避免重复写inertial -->
+    <xacro:macro name="gripper_link_inertial">
+        <inertial>
+            <!-- 惯性原点：质心位置，这里简化设置在连杆坐标系原点 -->
+            <origin xyz="0 0 0.0" rpy="0 0 0"/>
+            <!-- 连杆质量，引用上面定义的变量 -->
+            <mass value="${gripper_link_mass}"/>
+            <!-- 惯性张量，非对角项全部置0，主轴对齐 -->
+            <inertia
+                ixx="${gripper_link_ixx}" ixy="0.0" ixz="0.0"
+                iyy="${gripper_link_iyy}" iyz="0.0"
+                izz="${gripper_link_izz}"/>
+        </inertial>
+    </xacro:macro>
+    <!-- ===================== 主宏：自适应夹爪 =====================
+    参数说明：
+      parent：父连杆名称（mycobot机械臂末端法兰link）
+      prefix：名称前缀，用于多实例夹爪、防止link/joint重名
+      origin：xacro插入块，用来定义夹爪相对于parent的位姿(xyz rpy)
+    调用示例：<xacro:adaptive_gripper parent="link6" prefix="my_" origin> <origin xyz="0 0 0.05" rpy="0 0 0"/> </origin>
+    -->
+    <xacro:macro name="adaptive_gripper" params="parent prefix *origin">
+        <!-- ========== 1.夹爪底座连杆 gripper_base ========== -->
+        <link name="${prefix}gripper_base">
+            <!-- 底座惯性参数，底座质量0.07kg，单独定义，不使用手指宏 -->
+            <inertial>
+                <origin xyz="0 0 0.0" rpy="0 0 0"/>
+                <mass value="0.07"/>
+                <inertia
+                    ixx="0.000010725" ixy="0.0" ixz="0.0"
+                    iyy="0.000014392" iyz="0.0"
+                    izz="0.000018517"/>
+            </inertial>
+            <!-- Visual 可视化模型：仅用于RViz显示，不参与碰撞仿真 -->
+            <visual>
+                <geometry>
+                    <!-- 加载dae网格模型，文件路径在mycobot_description包下 -->
+                    <mesh filename="file://$(find mycobot_description)/meshes/adaptive_gripper/visual/gripper_base.dae"/>
+                </geometry>
+                <!-- 网格模型相对于link坐标系的偏移位姿 -->
+                <origin xyz="0.0 0.0 -0.012" rpy="0 0 0"/>
+            </visual>
+            <!-- Collision 碰撞模型：Gazebo碰撞检测用，一般用简化box代替精细mesh，提升仿真速度 -->
+            <collision>
+                <geometry>
+                    <!-- 简化包围盒：长宽高 0.065m ×0.025m ×0.025m -->
+                    <box size="0.065 0.025 0.025"/>
+                </geometry>
+                <origin xyz="0.0 0.0 0.0" rpy="0 0 0"/>
+            </collision>
+        </link>
+        <!-- 固定关节：机械臂末端法兰(parent) 固定连接 夹爪底座gripper_base -->
+        <joint name="${prefix}${parent}_to_${prefix}gripper_base" type="fixed">
+            <parent link="${prefix}${parent}"/>
+            <child link="${prefix}gripper_base"/>
+            <!-- 插入外部传入的origin位姿，宏调用时传入 -->
+            <xacro:insert_block name="origin"/>
+        </joint>
+        <!-- ========== 左侧手指三段连杆 ========== -->
+        <!-- left1：左手指最外侧指尖段 -->
+        <link name="${prefix}gripper_left1">
+            <!-- 复用惯性宏，快速填入质量惯量 -->
+            <xacro:gripper_link_inertial/>
+            <visual>
+                <geometry>
+                    <mesh filename="file://$(find mycobot_description)/meshes/adaptive_gripper/visual/gripper_left1.dae"/>
+                </geometry>
+                <origin xyz="0.039 -0.0133 -0.012" rpy="0 0 0"/>
+            </visual>
+            <collision>
+                <geometry>
+                    <box size="0.013 0.02 0.015"/>
+                </geometry>
+                <origin xyz="0.013 0.042 -0.010" rpy="0 0 0"/>
+            </collision>
+        </link>
+        <!-- left2：左手指中间段 -->
+        <link name="${prefix}gripper_left2">
+            <xacro:gripper_link_inertial/>
+            <visual>
+                <geometry>
+                    <mesh filename="file://$(find mycobot_description)/meshes/adaptive_gripper/visual/gripper_left2.dae"/>
+                </geometry>
+                <origin xyz="0.005 -0.0195 -0.012" rpy="0 0 0"/>
+            </visual>
+            <collision>
+                <geometry>
+                    <box size="0.02 0.02 0.02"/>
+                </geometry>
+                <origin xyz="-0.025 0.0 -0.010" rpy="0 0 0"/>
+            </collision>
+        </link>
+        <!-- left3：左手指根部段（主动关节所在连杆） -->
+        <link name="${prefix}gripper_left3">
+            <xacro:gripper_link_inertial/>
+            <visual>
+                <geometry>
+                    <mesh filename="file://$(find mycobot_description)/meshes/adaptive_gripper/visual/gripper_left3.dae"/>
+                </geometry>
+                <origin xyz="0.012 0.0025 -0.012" rpy="0 0 0"/>
+            </visual>
+            <collision>
+                <geometry>
+                    <box size="0.01 0.01 0.01"/>
+                </geometry>
+                <origin xyz="-0.014 0.005 0.005" rpy="0 0 0"/>
+            </collision>
+        </link>
+        <!-- ========== 右侧手指三段连杆 ========== -->
+        <!-- right1：右手指最外侧指尖段 -->
+        <link name="${prefix}gripper_right1">
+            <xacro:gripper_link_inertial/>
+            <visual>
+                <geometry>
+                    <mesh filename="file://$(find mycobot_description)/meshes/adaptive_gripper/visual/gripper_right1.dae"/>
+                </geometry>
+                <origin xyz="-0.039 -0.0133 -0.012" rpy="0 0 0"/>
+            </visual>
+            <collision>
+                <geometry>
+                    <box size="0.013 0.02 0.015"/>
+                </geometry>
+                <origin xyz="-0.013 0.042 -0.010" rpy="0 0 0"/>
+            </collision>
+        </link>
+        <!-- right2：右手指中间段 -->
+        <link name="${prefix}gripper_right2">
+            <xacro:gripper_link_inertial/>
+            <visual>
+                <geometry>
+                    <mesh filename="file://$(find mycobot_description)/meshes/adaptive_gripper/visual/gripper_right2.dae"/>
+                </geometry>
+                <origin xyz="-0.005 -0.0195 -0.012" rpy="0 0 0"/>
+            </visual>
+            <collision>
+                <geometry>
+                    <box size="0.02 0.02 0.02"/>
+                </geometry>
+                <origin xyz="0.025 0.0 -0.010" rpy="0 0 0"/>
+            </collision>
+        </link>
+        <!-- right3：右手指根部段 -->
+        <link name="${prefix}gripper_right3">
+            <xacro:gripper_link_inertial/>
+            <visual>
+                <geometry>
+                    <mesh filename="file://$(find mycobot_description)/meshes/adaptive_gripper/visual/gripper_right3.dae"/>
+                </geometry>
+                <origin xyz="-0.012 0.0025 -0.012" rpy="0 0 0"/>
+            </visual>
+            <collision>
+                <geometry>
+                    <box size="0.01 0.01 0.01"/>
+                </geometry>
+                <origin xyz="0.014 0.005 0.005" rpy="0 0 0"/>
+            </collision>
+        </link>
+        <!-- ===================== 关节定义（核心：1个主动关节 + 5个mimic随动关节） ===================== -->
+        <!-- 【唯一主动驱动关节】夹爪控制器关节，ros2_control只需要控制这一个关节 -->
+        <joint name="${prefix}gripper_controller" type="revolute">
+            <axis xyz="0 0 1"/> <!-- 旋转轴：Z轴，绕Z转动 -->
+            <!-- limit：关节限位，effort最大力矩，lower/upper角度范围(rad)，velocity最大速度 -->
+            <limit effort="${joint_effort}" lower="-0.7" upper="0.15" velocity="${joint_velocity}"/>
+            <parent link="${prefix}gripper_base"/>
+            <child link="${prefix}gripper_left3"/>
+            <origin xyz="-0.012 0.005 0" rpy="0 0 0"/>
+            <!-- 关节动力学参数：阻尼、摩擦 -->
+            <dynamics damping="${joint_damping}" friction="${joint_friction}"/>
+        </joint>
+        <!-- 左手指中间段left2：mimic跟随主动关节，multiplier=1，角度同步同方向 -->
+        <joint name="${prefix}gripper_base_to_${prefix}gripper_left2" type="revolute">
+            <axis xyz="0 0 1"/>
+            <limit effort="${joint_effort}" lower="-0.8" upper="0.5" velocity="${joint_velocity}"/>
+            <parent link="${prefix}gripper_base"/>
+            <child link="${prefix}gripper_left2"/>
+            <origin xyz="-0.005 0.027 0" rpy="0 0 0"/>
+            <!-- mimic：复刻关节，角度 = multiplier * 参考关节角度 + offset -->
+            <mimic joint="${prefix}gripper_controller" multiplier="1.0" offset="0"/>
+            <dynamics damping="${joint_damping}" friction="${joint_friction}"/>
+        </joint>
+        <!-- left3 -> left1指尖关节：multiplier=-1，反向跟随，实现连杆耦合折叠 -->
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