Commit message: Gazebo

File: src/mycobot_ros2/mycobot_description/urdf/mech/g_shape_base_v2_0.urdf.xacro (robot description, xacro)
@@ -1,45 +1,20 @@
 <?xml version="1.0" ?>
-<!--
-    声明这是一个 Xacro 文件。
-    Xacro 是 ROS 中用于生成 URDF 的 XML 宏语言，
-    可以通过 macro、参数、变量等方式复用机器人模型代码。
--->
 <robot xmlns:xacro="http://wiki.ros.org/xacro">
     <!--
         定义一个名为 g_shape_base 的 Xacro 宏。
         参数：
-        1. base_link：基础 Link 的名称，例如 base_link
-        2. prefix：Link 名称前缀，例如 robot1_、robot2_
-        调用这个宏后，会生成：
-            <link name="${prefix}${base_link}">
-        例如：
-            prefix = robot1_
-            base_link = base_link
-        最终 Link 名称就是：
-            robot1_base_link
+        1. base_link：基础 Link 的名称
+        2. prefix：Link 名称前缀
     -->
     <xacro:macro name="g_shape_base" params="base_link prefix">
-        <!--
-            定义机器人底座的 Link。
-            ${prefix}${base_link}
-            表示把 prefix 和 base_link 拼接起来。
-            例如：
-                prefix = ""
-                base_link = base_link
-                -> base_link
-            或：
-                prefix = robot1_
-                base_link = base_link
-                -> robot1_base_link
-        -->
+        <!-- 定义机器人底座的 Link -->
         <link name="${prefix}${base_link}">
             <!--
-                inertial：定义这个 Link 的动力学 / 惯性属性。
+                1. inertial：定义这个 Link 的动力学 / 惯性属性。
                 Gazebo 进行物理仿真时，需要知道物体的：
                 - 质量
                 - 质心位置
                 - 惯性矩阵
-                如果机器人需要在 Gazebo 中进行真实物理运动，
-                inertial 信息非常重要。
+                如果机器人需要在 Gazebo 中进行真实物理运动，inertial 信息非常重要。
             -->
             <inertial>
@@ -54,13 +29,10 @@
                 <!--
                     定义这个 Link 的质量。
-                    单位：
-                        kg
-                    这里表示底座质量为：
-                        0.33 kg
+                    单位：kg
+                    这里表示底座质量为：0.33 kg
                 -->
                 <mass value="0.33"/>
                 <!--
-                    定义惯性张量。
-                    惯性张量描述物体对于绕不同坐标轴旋转的惯性。
+                    定义惯性张量: 描述物体对于绕不同坐标轴旋转的惯性。
                     矩阵形式为：
                         | ixx  ixy  ixz |
@@ -71,24 +43,17 @@
                         iyy：绕 Y 轴的转动惯量
                         izz：绕 Z 轴的转动惯量
-                        ixy、ixz、iyz：
-                        表示不同坐标轴之间的惯性耦合项。
-                    单位通常为：
-                        kg·m²
+                        ixy、ixz、iyz：表示不同坐标轴之间的惯性耦合项。
+                    单位通常为：kg·m²
                 -->
                 <inertia
                     ixx="0.000784" ixy="0.0" ixz="0.0"
-                    iyy="0.000867" iyz="0.0"
-                    izz="0.001598"/>
+                    iyy="0.000867" iyz="0.0" izz="0.001598"/>
             </inertial>
             <!--
-                visual：定义机器人在 RViz / Gazebo 中
-                "看起来是什么样子"。
-                visual 主要负责显示模型，
-                不直接决定物理碰撞。
+                2. visual：定义机器人在 RViz / Gazebo 中 "看起来是什么样子"。
+                visual 主要负责显示模型，不直接决定物理碰撞。
             -->
             <visual>
-                <!--
-                    geometry：定义可视化几何形状。
-                -->
+                <!-- geometry：定义可视化几何形状 -->
                 <geometry>
                     <!--
@@ -132,5 +97,5 @@
             </visual>
             <!--
-                collision：定义这个 Link 用于物理碰撞检测的几何模型。
+                3. collision：定义这个 Link 用于物理碰撞检测的几何模型。
                 它和 visual 是分开的：
                     visual
@@ -171,5 +136,5 @@
         </link>
         <!--
-            gazebo：Gazebo 专用配置。
+            4. gazebo：Gazebo 专用配置。
             reference="${prefix}${base_link}"
             表示：

File: src/mycobot_ros2/mycobot_description/urdf/mech/mycobot_280_arm.urdf.xacro (robot description, xacro)
@@ -1,292 +1,416 @@
 <?xml version="1.0"?>
 <robot xmlns:xacro="http://www.ros.org/wiki/xacro">
-  <!-- xacro 内部变量 -->
-  <!-- 1. 关节最大力矩(N·m)，用于 joint limit 限制 -->
-  <xacro:property name="joint_effort" value="56.0"/>
-  <!-- 2. 关节最大角速度(rad/s)，用于 joint limit 限制 -->
-  <xacro:property name="joint_velocity" value="2.792527"/>
-  <!-- 3. 关节阻尼系数，Gazebo 动力学 dynamics 标签使用 -->
-  <xacro:property name="joint_damping" value="0.0"/>
-  <!-- 4. 关节库伦摩擦系数，Gazebo 动力学 dynamics 标签使用 -->
-  <xacro:property name="joint_friction" value="0.0"/>
-  <!-- 1. 连杆 1 质量，单位 kg，用于 inertial 惯性参数 -->
-  <xacro:property name="link1_mass" value="0.12"/>
-  <!-- 2. 连杆 2 质量，单位 kg，用于 inertial 惯性参数 -->
-  <xacro:property name="link2_mass" value="0.19"/>
-  <!-- 3. 连杆 3 质量，单位 kg，用于 inertial 惯性参数 -->
-  <xacro:property name="link3_mass" value="0.16"/>
-  <!-- 4. 连杆 4 质量，单位 kg，用于 inertial 惯性参数 -->
-  <xacro:property name="link4_mass" value="0.124"/>
-  <!-- 5. 连杆 5 质量，单位 kg，用于 inertial 惯性参数 -->
-  <xacro:property name="link5_mass" value="0.11"/>
-  <!-- 6. 连杆 6 质量，单位 kg，用于 inertial 惯性参数 -->
-  <xacro:property name="link6_mass" value="0.0739"/>
-  <!-- 7. 末端法兰 质量，单位 kg，用于 inertial 惯性参数 -->
-  <xacro:property name="flange_mass" value="0.035"/>
-  <!-- 定义宏：生成连杆惯性块，快速复用 inertial 标签 -->
-  <xacro:macro name="link_inertial" params="mass ixx iyy izz">
-    <!-- 惯性参数块，Gazebo 物理仿真必需，描述连杆质量与惯量 -->
-    <inertial>
-      <!-- 惯性坐标系原点，相对于连杆本体坐标系，rpy 姿态角 -->
-      <origin xyz="0 0 0.0" rpy="0 0 0"/>
-      <!-- 连杆质量 -->
-      <mass value="${mass}"/>
-      <!-- 惯性张量矩阵，简化模型：非对角惯量 ixy,ixz,iyz 全部置 0 -->
-      <inertia
-        ixx="${ixx}" ixy="0.0" ixz="0.0"
-        iyy="${iyy}" iyz="0.0"
-        izz="${izz}"/>
-    </inertial>
-  </xacro:macro>
-  <!-- 定义宏：给Gazebo中指定连杆设置视觉材质（仅Gazebo仿真生效，不影响URDF可视化） -->
-  <!-- 参数：
-     ref_link: 目标连杆名称，gazebo标签的reference，指定要修改材质的link
-     ambient: 环境光颜色，RGBA四元组，取值0~1
-     diffuse: 漫反射颜色，RGBA四元组，物体本身基础颜色
-     specular: 高光反射颜色，RGBA四元组，控制反光亮点颜色
-  -->
-  <xacro:macro name="material_visual" params="ref_link ambient diffuse specular">
-    <!-- Gazebo专属标签，reference指定作用的link，只在Gazebo仿真器识别 -->
-    <gazebo reference="${ref_link}">
-      <!-- Gazebo内的视觉渲染配置，和URDF的visual相互独立 -->
-      <visual>
-        <!-- 材质定义块 -->
-        <material>
-          <!-- 环境光颜色，环境照射到物体上的基础底色 RGBA -->
-          <ambient>${ambient}</ambient>
-          <!-- 漫反射颜色，物体受光呈现的主体颜色 RGBA -->
-          <diffuse>${diffuse}</diffuse>
-          <!-- 高光颜色，光源直射产生的反光亮点 RGBA -->
-          <specular>${specular}</specular>
-        </material>
-      </visual>
-    </gazebo>
-  </xacro:macro>
-  <!-- 定义宏：Mycobot280机械臂主体模型，批量生成所有连杆+关节，支持多实例前缀、自定义底座与末端法兰 -->
-  <!-- 参数说明：
-       base_link: 底座连杆名称，作为机械臂根部父连杆
-       flange_link: 末端法兰连杆名称
-       prefix: 连杆/关节名称前缀，用于在同一个urdf中加载多台机械臂，避免命名冲突
-       *origin: 可变参数块，用于传入固定关节的origin标签，适配底座安装位姿
-  -->
-  <xacro:macro name="mycobot_280_arm" params="base_link flange_link prefix *origin">
-    <!-- 1号连杆 -->
-    <link name="${prefix}link1">
-      <!-- 调用惯性宏，填入link1质量与惯量张量对角元 -->
-      <xacro:link_inertial mass="${link1_mass}" ixx="0.000148" iyy="0.000148" izz="0.000096"/>
-      <!-- RViz可视化几何体 -->
-      <visual>
-        <!-- 使用dae网格模型作为外观 -->
-        <geometry>
-          <mesh filename="file://$(find mycobot_description)/meshes/mycobot_280/visual/link1.dae"/>
-        </geometry>
-        <!-- 网格相对于link本体坐标系的偏移与旋转 -->
-        <origin xyz="0.0 0 0" rpy="0 0 ${-pi/2}"/>
-      </visual>
-      <!-- 碰撞检测几何体(Gazebo/碰撞检测用，简化包围盒，比mesh快很多) -->
-      <collision>
-        <geometry>
-          <box size="0.08 0.12 0.075"/>
-        </geometry>
-        <!-- 碰撞包围盒相对于link本体坐标系的位姿 -->
-        <origin xyz="0.0 -0.01 0.034" rpy="0 0 0"/>
-      </collision>
-    </link>
-    <!-- 2号连杆 -->
-    <link name="${prefix}link2">
-      <!-- 调用惯性宏，填入link2质量与惯量张量对角元 -->
-      <xacro:link_inertial mass="${link2_mass}" ixx="0.000148" iyy="0.000148" izz="0.000096"/>
-      <!-- RViz可视化几何体 -->
-      <visual>
-        <geometry>
-          <mesh filename="file://$(find mycobot_description)/meshes/mycobot_280/visual/link2.dae"/>
-        </geometry>
-        <origin xyz="0.0 0 -0.06096" rpy="0 0 ${-pi/2}"/>
-      </visual>
-      <!-- 碰撞几何体：圆柱简化包围体 -->
-      <collision>
-        <geometry>
-          <cylinder radius="0.025" length="0.085"/>
-        </geometry>
-        <origin xyz="0.0 0 -0.02" rpy="0 0 ${-pi/2}"/>
-      </collision>
-    </link>
-    <!-- 3号连杆 -->
-    <link name="${prefix}link3">
-      <!-- 调用惯性宏，填入link3质量与惯量张量对角元 -->
-      <xacro:link_inertial mass="${link3_mass}" ixx="0.000148" iyy="0.000148" izz="0.000096"/>
-      <!-- RViz可视化几何体 -->
-      <visual>
-        <geometry>
-          <mesh filename="file://$(find mycobot_description)/meshes/mycobot_280/visual/link3.dae"/>
-        </geometry>
-        <origin xyz="0.0 0 0.03256" rpy="0 ${-pi/2} 0"/>
-      </visual>
-      <!-- 碰撞几何体：圆柱简化包围体 -->
-      <collision>
-        <geometry>
-          <cylinder radius="0.025" length="0.15"/>
-        </geometry>
-        <origin xyz="-0.058 0 0.059" rpy="0 ${-pi/2} 0"/>
-      </collision>
-    </link>
-    <!-- 4号连杆 -->
-    <link name="${prefix}link4">
-      <!-- 调用惯性宏，填入link4质量与惯量张量对角元 -->
-      <xacro:link_inertial mass="${link4_mass}" ixx="0.000103" iyy="0.000103" izz="0.000096"/>
-      <!-- RViz可视化几何体 -->
-      <visual>
-        <geometry>
-          <mesh filename="file://$(find mycobot_description)/meshes/mycobot_280/visual/link4.dae"/>
-        </geometry>
-        <origin xyz="0.0 0 0.03056" rpy="0 ${-pi/2} 0"/>
-      </visual>
-      <!-- 碰撞几何体：圆柱简化包围体 -->
-      <collision>
-        <geometry>
-          <cylinder radius="0.025" length="0.125"/>
-        </geometry>
-        <origin xyz="-0.05 0 0.0" rpy="0 ${-pi/2} 0"/>
-      </collision>
-    </link>
-    <!-- 5号连杆 -->
-    <link name="${prefix}link5">
-      <!-- 调用惯性宏，填入link5质量与惯量张量对角元 -->
-      <xacro:link_inertial mass="${link5_mass}" ixx="0.000103" iyy="0.000103" izz="0.000096"/>
-      <!-- RViz可视化几何体 -->
-      <visual>
-        <geometry>
-          <mesh filename="file://$(find mycobot_description)/meshes/mycobot_280/visual/link5.dae"/>
-        </geometry>
-        <origin xyz="0.0 0 -0.03356" rpy="${-pi/2} 0 0"/>
-      </visual>
-      <!-- 碰撞几何体：长方体包围盒 -->
-      <collision>
-        <geometry>
-          <box size="0.03 0.035 0.05"/>
-        </geometry>
-        <origin xyz="0.0 0 -0.005" rpy="0 0.0 0"/>
-      </collision>
-    </link>
-    <!-- 6号连杆 -->
-    <link name="${prefix}link6">
-      <!-- 调用惯性宏，填入link6质量与惯量张量对角元 -->
-      <xacro:link_inertial mass="${link6_mass}" ixx="0.00006649" iyy="0.00006649" izz="0.000096"/>
-      <!-- RViz可视化几何体 -->
-      <visual>
-        <geometry>
-          <mesh filename="file://$(find mycobot_description)/meshes/mycobot_280/visual/link6.dae"/>
-        </geometry>
-        <origin xyz="0 0.00 -0.038" rpy="0 0 0"/>
-      </visual>
-      <!-- 碰撞几何体：圆柱简化包围体 -->
-      <collision>
-        <geometry>
-          <cylinder radius="0.025" length="0.06"/>
-        </geometry>
-        <origin xyz="0 0.00 0.0" rpy="${-pi/2} 0 0"/>
-      </collision>
-    </link>
-    <!-- 末端法兰连杆 -->
-    <link name="${prefix}${flange_link}">
-      <!-- 调用惯性宏，填入末端法兰质量与惯量张量对角元 -->
-      <xacro:link_inertial mass="${flange_mass}" ixx="0.0000149" iyy="0.0000149" izz="0.0000196"/>
-      <!-- RViz可视化几何体 -->
-      <visual>
-        <geometry>
-          <mesh filename="file://$(find mycobot_description)/meshes/mycobot_280/visual/link7.dae"/>
-        </geometry>
-        <origin xyz="0.0 0 -0.012" rpy="0 0 0"/>
-      </visual>
-      <!-- 碰撞几何体：小圆柱包围体 -->
-      <collision>
-        <geometry>
-          <cylinder radius="0.02" length="0.02"/>
-        </geometry>
-        <origin xyz="0 0.00 0.0" rpy="0 0 0"/>
-      </collision>
-    </link>
-    <!-- 底座到link1固定关节，用于把机械臂挂载到基座上 -->
-    <joint name="${prefix}${base_link}_to_${prefix}link1" type="fixed">
-      <!-- 父连杆：底座 -->
-      <parent link="${prefix}${base_link}"/>
-      <!-- 子连杆：1号连杆 -->
-      <child link="${prefix}link1"/>
-      <!-- 插入外部传入的origin块，自定义底座安装偏移 -->
-      <xacro:insert_block name="origin"/>
-    </joint>
-    <!-- J1：link1 -> link2 旋转关节，机械臂第1个转动轴 -->
-    <joint name="${prefix}link1_to_${prefix}link2" type="revolute">
-      <!-- 旋转轴方向向量，在父连杆坐标系下 -->
-      <axis xyz="0 0 1"/>
-      <!-- 关节限位：最大力矩、角度上下限、最大角速度 -->
-      <limit effort="${joint_effort}" lower="-2.879793" upper="2.879793" velocity="${joint_velocity}"/>
-      <parent link="${prefix}link1"/>
-      <child link="${prefix}link2"/>
-      <!-- 子连杆相对于父连杆的位姿 -->
-      <origin xyz="0 0 0.13156" rpy="0 0 ${pi/2}"/>
-      <!-- 动力学参数：阻尼、库伦摩擦，Gazebo仿真使用 -->
-      <dynamics damping="${joint_damping}" friction="${joint_friction}"/>
-    </joint>
-    <!-- J2：link2 -> link3 旋转关节，机械臂第2个转动轴 -->
-    <joint name="${prefix}link2_to_${prefix}link3" type="revolute">
-      <axis xyz="0 0 1"/>
-      <limit effort="${joint_effort}" lower="-2.879793" upper="2.879793" velocity="${joint_velocity}"/>
-      <parent link="${prefix}link2"/>
-      <child link="${prefix}link3"/>
-      <origin xyz="0 0 -0.001" rpy="0 ${pi/2} ${-pi/2}"/>
-      <dynamics damping="${joint_damping}" friction="${joint_friction}"/>
-    </joint>
-    <!-- J3：link3 -> link4 旋转关节，机械臂第3个转动轴 -->
-    <joint name="${prefix}link3_to_${prefix}link4" type="revolute">
-      <axis xyz="0 0 1"/>
-      <limit effort="${joint_effort}" lower="-2.879793" upper="2.879793" velocity="${joint_velocity}"/>
-      <parent link="${prefix}link3"/>
-      <child link="${prefix}link4"/>
-      <origin xyz="-0.1104 0 0" rpy="0 0 0"/>
-      <dynamics damping="${joint_damping}" friction="${joint_friction}"/>
-    </joint>
-    <!-- J4：link4 -> link5 旋转关节，机械臂第4个转动轴 -->
-    <joint name="${prefix}link4_to_${prefix}link5" type="revolute">
-      <axis xyz="0 0 1"/>
-      <limit effort="${joint_effort}" lower="-2.879793" upper="2.879793" velocity="${joint_velocity}"/>
-      <parent link="${prefix}link4"/>
-      <child link="${prefix}link5"/>
-      <origin xyz="-0.096 0 0.06062" rpy="0 0 ${-pi/2}"/>
-      <dynamics damping="${joint_damping}" friction="${joint_friction}"/>
-    </joint>
-    <!-- J5：link5 -> link6 旋转关节，机械臂第5个转动轴 -->
-    <joint name="${prefix}link5_to_${prefix}link6" type="revolute">
-      <axis xyz="0 0 1"/>
-      <limit effort="${joint_effort}" lower="-2.879793" upper="2.879793" velocity="${joint_velocity}"/>
-      <parent link="${prefix}link5"/>
-      <child link="${prefix}link6"/>
-      <origin xyz="0 -0.07318 0" rpy="${pi/2} ${-pi/2} 0"/>
-      <dynamics damping="${joint_damping}" friction="${joint_friction}"/>
-    </joint>
-    <!-- J6：link6 -> 末端法兰 旋转关节，机械臂第6个转动轴 -->
-    <joint name="${prefix}link6_to_${prefix}${flange_link}" type="revolute">
-      <axis xyz="0 0 1"/>
-      <!-- J6单独角度限位，和前面J1~J5范围不同 -->
-      <limit effort="${joint_effort}" lower="-3.05" upper="3.05" velocity="${joint_velocity}"/>
-      <parent link="${prefix}link6"/>
-      <child link="${prefix}${flange_link}"/>
-      <origin xyz="0 0.0456 0" rpy="${-pi/2} 0 0"/>
-      <dynamics damping="${joint_damping}" friction="${joint_friction}"/>
-    </joint>
-    <!-- 调用材质宏：Gazebo渲染，设置link1材质颜色 -->
-    <xacro:material_visual ref_link="${prefix}link1" ambient="0.5 0.5 0.5 1" diffuse="0.5 0.5 0.5 1" specular="0.5 0.5 0.5 1"/>
-    <!-- 调用材质宏：Gazebo渲染，设置link2材质颜色 -->
-    <xacro:material_visual ref_link="${prefix}link2" ambient="1 1 1 1" diffuse="1 1 1 1" specular="1 1 1 1"/>
-    <!-- 调用材质宏：Gazebo渲染，设置link3材质颜色 -->
-    <xacro:material_visual ref_link="${prefix}link3" ambient="1 1 1 1" diffuse="1 1 1 1" specular="1 1 1 1"/>
-    <!-- 调用材质宏：Gazebo渲染，设置link4材质颜色 -->
-    <xacro:material_visual ref_link="${prefix}link4" ambient="1 1 1 1" diffuse="1 1 1 1" specular="1 1 1 1"/>
-    <!-- 调用材质宏：Gazebo渲染，设置link5材质颜色 -->
-    <xacro:material_visual ref_link="${prefix}link5" ambient="1 1 1 1" diffuse="1 1 1 1" specular="1 1 1 1"/>
-    <!-- 调用材质宏：Gazebo渲染，设置link6材质颜色 -->
-    <xacro:material_visual ref_link="${prefix}link6" ambient="1 1 1 1" diffuse="1 1 1 1" specular="1 1 1 1"/>
-    <!-- 调用材质宏：Gazebo渲染，设置末端法兰材质颜色 -->
-    <xacro:material_visual ref_link="${prefix}${flange_link}" ambient="0.5 0.5 0.5 1" diffuse="0.5 0.5 0.5 1" specular="0.5 0.5 0.5 1"/>
-  </xacro:macro>
+    <!-- xacro 内部变量 -->
+    <!-- 1. 关节最大力矩(N·m)，用于 joint limit 限制 -->
+    <xacro:property name="joint_effort" value="56.0"/>
+    <!-- 2. 关节最大角速度(rad/s)，用于 joint limit 限制 -->
+    <xacro:property name="joint_velocity" value="2.792527"/>
+    <!-- 3. 关节阻尼系数，Gazebo 动力学 dynamics 标签使用 -->
+    <xacro:property name="joint_damping" value="0.0"/>
+    <!-- 4. 关节库伦摩擦系数，Gazebo 动力学 dynamics 标签使用 -->
+    <xacro:property name="joint_friction" value="0.0"/>
+    <!-- 1. 连杆 1 质量，单位 kg，用于 inertial 惯性参数 -->
+    <xacro:property name="link1_mass" value="0.12"/>
+    <!-- 2. 连杆 2 质量，单位 kg，用于 inertial 惯性参数 -->
+    <xacro:property name="link2_mass" value="0.19"/>
+    <!-- 3. 连杆 3 质量，单位 kg，用于 inertial 惯性参数 -->
+    <xacro:property name="link3_mass" value="0.16"/>
+    <!-- 4. 连杆 4 质量，单位 kg，用于 inertial 惯性参数 -->
+    <xacro:property name="link4_mass" value="0.124"/>
+    <!-- 5. 连杆 5 质量，单位 kg，用于 inertial 惯性参数 -->
+    <xacro:property name="link5_mass" value="0.11"/>
+    <!-- 6. 连杆 6 质量，单位 kg，用于 inertial 惯性参数 -->
+    <xacro:property name="link6_mass" value="0.0739"/>
+    <!-- 7. 末端法兰 质量，单位 kg，用于 inertial 惯性参数 -->
+    <xacro:property name="flange_mass" value="0.035"/>
+    <!--
+        1. 宏定义: 生成连杆惯性块
+        参数:
+            1) mass: 质量, 表示这个 Link 有多重, kg
+            2) ixx: 绕 x轴 的转动惯量, 表示绕 x 轴转有多难, kg·m²
+            2) iyy: 绕 y轴 的转动惯量, 表示绕 y 轴转有多难, kg·m²
+            2) izz: 绕 z轴 的转动惯量, 表示绕 z 轴转有多难, kg·m²
+    -->
+    <xacro:macro name="link_inertial" params="mass ixx iyy izz">
+        <!-- 连杆惯性块 -->
+        <inertial>
+            <!-- 1. 惯性坐标系 相对于 连杆坐标系 的 位置 和 位姿 -->
+            <origin xyz="0.0 0.0 0.0" rpy="0.0 0.0 0.0"/>
+            <!-- 2. 连杆质量(kg) -->
+            <mass value="${mass}"/>
+            <!-- 3. 惯性张量矩阵 -->
+            <inertia
+                ixx="${ixx}" ixy="0.0" ixz="0.0"
+                iyy="${iyy}" iyz="0.0" izz="${izz}"
+            />
+        </inertial>
+    </xacro:macro>
+    <!-- 2. 宏定义: 给 Gazebo 中指定连杆设置视觉材质(仅在Gazebo中生效) -->
+    <!--
+        参数:
+            1) ref_link: 指定要修改的目标连杆名称
+            2）ambient: 环境光颜色, RGBA
+            3）diffuse: 漫反射颜色, RGBA
+            4）specular: 高光反射颜色, RGBA
+    -->
+    <xacro:macro name="material_visual" params="ref_link ambient diffuse specular">
+        <!-- 指定 Gazebo 渲染的 连杆 -->
+        <gazebo reference="${ref_link}">
+            <!-- Gazebo 视觉渲染配置, 和 URDF 的 visual 相互独立 -->
+            <visual>
+                <!-- 材质定义 -->
+                <material>
+                    <!-- 环境光颜色，环境照射到物体上的基础底色 RGBA -->
+                    <ambient>${ambient}</ambient>
+                    <!-- 漫反射颜色，物体受光呈现的主体颜色 RGBA -->
+                    <diffuse>${diffuse}</diffuse>
+                    <!-- 高光颜色，光源直射产生的反光亮点 RGBA -->
+                    <specular>${specular}</specular>
+                </material>
+            </visual>
+        </gazebo>
+    </xacro:macro>
+    <!-- 3. 宏定义: 批量生成 link & joint  -->
+    <xacro:macro name="mycobot_280_arm" params="base_link flange_link prefix *origin">
+        <!-- 1 号连杆 -->
+        <link name="${prefix}link1">
+            <!-- 1) 调用惯性宏定义 -->
+            <xacro:link_inertial
+                mass="${link1_mass}"
+                ixx="0.000148" iyy="0.000148" izz="0.000096"
+            />
+            <!-- 2) 可视化 -->
+            <visual>
+                <!-- 使用 dae 网络模型 -->
+                <geometry>
+                    <mesh filename="file://$(find mycobot_description)/meshes/mycobot_280/visual/link1.dae" />
+                </geometry>
+                <!-- 定位 -->
+                <origin xyz="0.0 0 0" rpy="0 0 ${-pi/2}"/>
+            </visual>
+            <!-- 3) 碰撞 -->
+            <collision>
+                <geometry>
+                    <box size="0.08 0.12 0.075"/>
+                </geometry>
+                <origin xyz="0.0 -0.01 0.034" rpy="0 0 0"/>
+            </collision>
+        </link>
+        <!-- 2 号连杆 -->
+        <link name="${prefix}link2">
+            <!-- 1) 调用惯性宏定义 -->
+            <xacro:link_inertial
+                mass="${link2_mass}"
+                ixx="0.000148" iyy="0.000148" izz="0.000096"
+            />
+            <!-- 2) 可视化 -->
+            <visual>
+                <!-- 使用 dae 网络模型 -->
+                <geometry>
+                    <mesh filename="file://$(find mycobot_description)/meshes/mycobot_280/visual/link2.dae" />
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
File: src/mycobot_ros2/mycobot_description/urdf/robots/mycobot_280.urdf.xacro (robot description, xacro)
@@ -60,4 +60,5 @@
         prefix="$(arg prefix)"
     >
+        <!-- block参数传给宏 -->
         <origin xyz="0.0 0.0 0.0" rpy="0.0 0.0 0.0"/>
     </xacro:mycobot_280_arm>
